Commit message: Controller

File: install/car_description/share/car_description/urdf/robot.urdf.xacro (robot description, xacro)
@@ -1,5 +1,7 @@
 <?xml version="1.0"?>
 <robot xmlns:xacro="http://www.ros.org/wiki/xacro" name="car">
+    <xacro:arg name="is_ignition" default="true"/>
     <xacro:include filename="$(find car_description)/urdf/robot_gazebo.xacro"/>
+    <xacro:include filename="$(find car_description)/urdf/robot_ros2_control.xacro"/>
     <link name="base_footprint"/>
     <link name="base_link">
@@ -20,5 +22,5 @@
         <origin xyz="0 0 0" rpy="0 0 0" />
         <geometry>
-            <mesh filename="package://bumperbot_description/meshes/base_link.STL" />
+            <mesh filename="package://car_description/meshes/base_link.STL" />
         </geometry>
         </collision>

File: install/car_description/share/car_description/urdf/robot_gazebo.xacro (robot description, xacro)
@@ -35,3 +35,8 @@
         <maxVel>1.0</maxVel>
     </gazebo>
+    <gazebo>
+        <plugin filename="gz_ros2_control-system" name="gz_ros2_control::GazeboSimROS2ControlPlugin">
+            <parameters>$(find car_controller)/config/car_controllers.yaml</parameters>
+        </plugin>
+    </gazebo>
 </robot>
