Commit message: IMU

File: src/car_description/urdf/robot.urdf.xacro (robot description, xacro)
@@ -139,3 +139,33 @@
         <axis xyz="0 0 0" />
     </joint>
+  <link name="imu_link">
+    <inertial>
+      <origin xyz="-0.00552433659106688 0.000168210391520346 0.000514000497342681" rpy="0 0 0" />
+      <mass value="0.000528415362211671" />
+      <inertia ixx="1.46176048428261E-08" ixy="1.40015117949421E-10" ixz="-1.99633872937403E-12"
+               iyy="8.59662482954888E-09" iyz="7.52375112767959E-12"
+               izz="2.30279421279312E-08" />
+    </inertial>
+    <visual>
+      <origin xyz="0 0 0" rpy="0 0 0" />
+      <geometry>
+        <mesh filename="package://car_description/meshes/imu_link.STL" />
+      </geometry>
+      <material name="">
+        <color rgba="0.792156862745098 0.819607843137255 0.933333333333333 1" />
+      </material>
+    </visual>
+    <collision>
+      <origin xyz="0 0 0" rpy="0 0 0" />
+      <geometry>
+        <mesh filename="package://car_description/meshes/imu_link.STL" />
+      </geometry>
+    </collision>
+  </link>
+    <joint name="imu_joint" type="fixed">
+        <origin xyz="0 0 0.07" rpy="0 0 0" />
+        <parent link="base_link" />
+        <child link="imu_link" />
+        <axis xyz="0 0 0" />
+    </joint>
 </robot>

File: src/car_description/urdf/robot_gazebo.xacro (robot description, xacro)
@@ -39,4 +39,56 @@
             <parameters>$(find car_controller)/config/car_controllers.yaml</parameters>
         </plugin>
+        <plugin filename="gz-sim-imu-system" name="gz::sim::systems::Imu">
+        </plugin>
+    </gazebo>
+    <gazebo reference="imu_link">
+        <sensor name="imu" type="imu">
+            <always_on>true</always_on>
+            <update_rate>100</update_rate>
+            <gz_frame_id>imu_link</gz_frame_id>
+            <topic>imu</topic>
+            <imu>
+            <angular_velocity>
+                <x>
+                    <noise type="gaussian">
+                        <mean>0.0</mean>
+                        <stddev>2e-4</stddev>
+                    </noise>
+                </x>
+                <y>
+                    <noise type="gaussian">
+                        <mean>0.0</mean>
+                        <stddev>2e-4</stddev>
+                    </noise>
+                </y>
+                <z>
+                    <noise type="gaussian">
+                        <mean>0.0</mean>
+                        <stddev>2e-4</stddev>
+                    </noise>
+                </z>
+            </angular_velocity>
+            <linear_acceleration>
+                <x>
+                    <noise type="gaussian">
+                        <mean>0.0</mean>
+                        <stddev>1.7e-2</stddev>
+                    </noise>
+                </x>
+                <y>
+                    <noise type="gaussian">
+                        <mean>0.0</mean>
+                        <stddev>1.7e-2</stddev>
+                    </noise>
+                </y>
+                <z>
+                    <noise type="gaussian">
+                        <mean>0.0</mean>
+                        <stddev>1.7e-2</stddev>
+                    </noise>
+                </z>
+            </linear_acceleration>
+            </imu>
+        </sensor>
     </gazebo>
 </robot>

Commit message: Lidar

File: src/car_description/urdf/robot.urdf.xacro (robot description, xacro)
@@ -169,3 +169,30 @@
         <axis xyz="0 0 0" />
     </joint>
+    <link name="laser_link">
+        <inertial>
+        <origin xyz="-0.011945780406062 -0.000381929217680526 -0.0170649378129477" rpy="0 0 0" />
+        <mass value="0.073084435549317" />
+        <inertia ixx="1.96074931730795E-05" ixy="-3.62091076640009E-07" ixz="4.28230084046735E-07"
+                iyy="2.40983835136327E-05" iyz="1.50180909250652E-08"
+                izz="4.14184164228595E-05" />
+        </inertial>
+        <visual>
+            <origin rpy="0 0 0" xyz="0 0 0"/>
+            <geometry>
+                <mesh filename="package://car_description/meshes/laser_link.STL"/>
+            </geometry>
+        </visual>
+        <collision>
+            <origin xyz="0 0 0" rpy="0 0 0" />
+            <geometry>
+                <mesh filename="package://car_description/meshes/laser_link.STL"/>
+            </geometry>
+        </collision>
+    </link>
+    <joint name="laser_joint" type="fixed">
+        <parent link="base_link"/>
+        <child link="laser_link"/>
+        <origin xyz="0 0 0.1208" rpy="0 0 3.14"/>
+        <axis xyz="0 0 0" />
+    </joint>
 </robot>

File: src/car_description/urdf/robot_gazebo.xacro (robot description, xacro)
@@ -40,4 +40,7 @@
         </plugin>
         <plugin filename="gz-sim-imu-system" name="gz::sim::systems::Imu">
+        </plugin>
+        <plugin filename="gz-sim-sensors-system" name="gz::sim::systems::Sensors">
+            <render_engine>ogre2</render_engine>
         </plugin>
     </gazebo>
@@ -92,3 +95,32 @@
         </sensor>
     </gazebo>
+    <gazebo reference="laser_link">
+        <sensor name="lidar" type="gpu_ray">
+            <always_on>true</always_on>
+            <visualize>true</visualize>
+            <topic>scan</topic>
+            <update_rate>5</update_rate>
+            <gz_frame_id>laser_link</gz_frame_id>
+            <ray>
+                <scan>
+                    <horizontal>
+                        <samples>360</samples>
+                        <resolution>1.0</resolution>
+                        <min_angle>0</min_angle>
+                        <max_angle>6.28</max_angle>
+                    </horizontal>
+                </scan>
+                <range>
+                    <min>0.12</min> <!-- cant detect less than 12 cm -->
+                    <max>12.0</max>
+                    <resolution>0.02</resolution>
+                </range>
+                <noise>
+                    <type>gaussian</type>
+                    <mean>0.0</mean>
+                    <stddev>0.01</stddev>
+                </noise>
+            </ray>
+        </sensor>
+    </gazebo>
 </robot>

Commit message: mLLM

File: src/car_description/urdf/robot.urdf.xacro (robot description, xacro)
@@ -196,3 +196,30 @@
         <axis xyz="0 0 0" />
     </joint>
+    <link name="camera_link">
+        <inertial>
+        <origin xyz="0.0 0.0 0.0" rpy="0 0 0" />
+        <mass value="0.05" />
+        <inertia ixx="1e-05" ixy="0.0" ixz="0.0"
+                iyy="1e-05" iyz="0.0"
+                izz="1e-05" />
+        </inertial>
+        <visual>
+            <origin rpy="0 0 0" xyz="0 0 0"/>
+            <geometry>
+                <box size="0.05 0.03 0.03"/>
+            </geometry>
+        </visual>
+        <collision>
+        <origin xyz="0 0 0" rpy="0 0 0" />
+            <geometry>
+                    <box size="0.05 0.03 0.03"/>
+            </geometry>
+        </collision>
+    </link>
+    <joint name="camera_joint" type="fixed">
+        <parent link="base_link"/>
+        <child link="camera_link"/>
+        <origin xyz="0 0 0.13" rpy="0 0 0"/>
+        <axis xyz="0 0 0" />
+    </joint>
 </robot>

File: src/car_description/urdf/robot_gazebo.xacro (robot description, xacro)
@@ -42,4 +42,7 @@
         </plugin>
         <plugin filename="gz-sim-sensors-system" name="gz::sim::systems::Sensors">
+            <render_engine>ogre2</render_engine>
+        </plugin>
+        <plugin filename="gz-sim-camera-system" name="gz::sim::systems::Camera">
             <render_engine>ogre2</render_engine>
         </plugin>
@@ -124,3 +127,30 @@
         </sensor>
     </gazebo>
+    <gazebo reference="camera_link">
+        <sensor name="camera" type="camera">
+            <always_on>true</always_on>
+            <update_rate>10</update_rate>
+            <gz_frame_id>camera_link</gz_frame_id>
+            <topic>camera</topic>
+            <image>
+                <width>640</width>
+                <height>480</height>
+                <format>R8G8B8</format>
+                <clip_near>0.1</clip_near>
+                <clip_far>10.0</clip_far>
+            </image>
+            <camera>
+                <horizontal_fov>1.047</horizontal_fov>
+                <image>
+                    <format>R8G8B8</format>
+                    <width>640</width>
+                    <height>480</height>
+                </image>
+                <clip>
+                    <near>0.1</near>
+                    <far>10.0</far>
+                </clip>
+            </camera>
+        </sensor>
+    </gazebo>
 </robot>
